File: FabPOx.brd (EAGLE design)
At the start: 68.6 x 40.6 mm, 37 parts, among them IC1 ATTINY44-SSU, IC2 OPAMPSO08, Q1 TRANSISTOR_PNPSMD, Q2 TRANSISTOR_PNPSMD, U1 HC_05

Commit message: Fixed value on capacitor C1
Parts:
- C1: value 220p -> 10u
